File: EAGLE/Board/Board.sch (EAGLE design)
At the start: 2 parts

Commit message: board
Parts:
- added CAP3, CAP5: 1uF, 433:CAP-CERAMIC
- added CAP4: 10uF, 433:CAP-TANTALUM
- added DEBUG, RESET: BUTTON, 433:BUTTON
- added GREEN: LED, 433:LED
- added J1: (no value), 433:CONNECTOR-5PINPTH
- added J2: USB-MINIB-5PIN, 433:USB-MINIB-5PIN
- added RES1, RES2: 10k, 433:RESISTOR
- added RES3: 330, 433:RESISTOR
Connections:
- removed net N$3: CONTROLLER.P19, CONTROLLER.P27, CONTROLLER.P8, RESONATOR.2
- removed net N$4: CONTROLLER.P13, CONTROLLER.P23, CONTROLLER.P28
- new net +3.3: CAP3.A, CAP5.A, CONTROLLER.P13, CONTROLLER.P23, CONTROLLER.P28, RES1.P$1, RES2.P$1
- new net GND: CAP3.B, CAP4.-, CAP5.B, CONTROLLER.P19, CONTROLLER.P27, CONTROLLER.P8, DEBUG.P$1, RES3.P$1, RESET.P$1, RESONATOR.2
- new net GREEN: CONTROLLER.P12, GREEN.+
- new net N$5: CAP4.+, CONTROLLER.P20
- new net N$6: GREEN.-, RES3.P$2
- new net N$7: CONTROLLER.P1\, RES1.P$2, RESET.P$2
- new net N$8: CONTROLLER.P11, DEBUG.P$2, RES2.P$2
Other:
- moved on the sheet: RESONATOR

Commit message: schematics ready
Parts:
- added CAP1: 1uF, 433:CAP-CERAMIC
- added CAP2: 10uF, 433:CAP-TANTALUM
- added IC1: REGULATORLMLZ, 433:REGULATORLMLZ
- added PICKIT-CONN: (no value), 433:CONNECTOR-5PINPTH
- added RED: ON-OFF, 433:LED
- added RES4: 330, 433:RESISTOR
- GREEN: value LED -> DEBUG
- J1: value (none) -> 2X6 FEMALE; device 433:CONNECTOR-5PINPTH -> 433:CONNECTOR-12PINPTH_FEMALE
- RES1: value 10k -> 330
- RES3: value 330 -> 10k
Connections:
- removed net GREEN: CONTROLLER.P12, GREEN.+
- removed net N$8: CONTROLLER.P11, DEBUG.P$2, RES2.P$2
- new net +5: CAP1.A, CONTROLLER.P15, IC1.VI, J2.VBUS
- new net N$3: RED.+, RES1.P$1
- new net N$4: CONTROLLER.P4, PICKIT-CONN.4
- new net N$9: CONTROLLER.P5, PICKIT-CONN.5
- new net RA0: CONTROLLER.P2, J1.1
- new net RA1: CONTROLLER.P3, J1.3
- new net RA4: CONTROLLER.P12, GREEN.+, J1.11
- new net RB13: CONTROLLER.P24, J1.6
- new net RB14: CONTROLLER.P25, J1.4
- new net RB15: CONTROLLER.P26, J1.2
- new net RB2: CONTROLLER.P6, J1.5
- new net RB3: CONTROLLER.P7, J1.7
- new net RB4: CONTROLLER.P11, DEBUG.P$2, J1.9, RES3.P$2
- new net RB7: CONTROLLER.P16, J1.12
- new net RB8: CONTROLLER.P17, J1.10
- new net RB9: CONTROLLER.P18, J1.8
- new net USB-D+: CONTROLLER.P21, J2.D+
- new net USB-D-: CONTROLLER.P22, J2.D-
- new net USB-ID: CONTROLLER.P14, J2.ID
- net +3.3: now also CAP2.+, IC1.VO, PICKIT-CONN.2, RES1.P$2, RES3.P$1; no longer RES1.P$1
- net GND: now also CAP1.B, CAP2.-, IC1.ADJ, J2.GND, PICKIT-CONN.3, RED.-, RES4.P$1; no longer CAP4.-, RES3.P$1
- net N$6: now also RES4.P$2; no longer RES3.P$2
- net N$7: now also PICKIT-CONN.1, RES2.P$2; no longer RES1.P$2
Other:
- moved on the sheet: CAP4, J2, RES1, RES2, RES3

Commit message: board
Parts:
- removed J1: 2X6 FEMALE, 433:CONNECTOR-12PINPTH_FEMALE
- added GPIO: (no value), 433:M08X2
- renumbered IC1 to 1702, J2 to USB
Connections:
- net +3.3: now also GPIO.2
- net +5: now also GPIO.4
- net GND: now also CAP4.-, GPIO.1, GPIO.3
- net RA0: now also GPIO.5; no longer J1.1
- net RA1: now also GPIO.7; no longer J1.3
- net RA4: now also GPIO.15; no longer J1.11
- net RB13: now also GPIO.10; no longer J1.6
- net RB14: now also GPIO.8; no longer J1.4
- net RB15: now also GPIO.6; no longer J1.2
- net RB2: now also GPIO.9; no longer J1.5
- net RB3: now also GPIO.11; no longer J1.7
- net RB4: now also GPIO.13; no longer J1.9
- net RB7: now also GPIO.16; no longer J1.12
- net RB8: now also GPIO.14; no longer J1.10
- net RB9: now also GPIO.12; no longer J1.8
Other:
- moved on the sheet: CAP4

Commit message: board
Parts:
- removed GPIO: (no value), 433:M08X2
- added GPIO1, GPIO2: (no value), 433:M08
- added U$1: SWITCH, 433:SWITCH
- RESONATOR: device 433:DIP-CERAMIC-RESONATOR/-OSCILLATOR-8MHZ(3P-2.5-8X3MM) -> 433:OSCILATOR-CRYSTAL
- USB: value USB-MINIB-5PIN -> USB-MINIB; device 433:USB-MINIB-5PIN -> 433:USB-MINIB
- renumbered CONTROLLER to PIC32-MX250F128B
Connections:
- new net N$8: U$1.IN, USB.VBUS
- net +3.3: now also GPIO1.7; no longer GPIO.2
- net +5: now also GPIO2.2, U$1.OA; no longer GPIO.4, USB.VBUS
- net GND: now also GPIO1.8, GPIO2.1; no longer GPIO.1, GPIO.3
- net RA0: now also GPIO1.1; no longer GPIO.5
- net RA1: now also GPIO1.2; no longer GPIO.7
- net RA4: now also GPIO1.6; no longer GPIO.15
- net RB13: now also GPIO2.6; no longer GPIO.10
- net RB14: now also GPIO2.7; no longer GPIO.8
- net RB15: now also GPIO2.8; no longer GPIO.6
- net RB2: now also GPIO1.3; no longer GPIO.9
- net RB3: now also GPIO1.4; no longer GPIO.11
- net RB4: now also GPIO1.5; no longer GPIO.13
- net RB7: now also GPIO2.3; no longer GPIO.16
- net RB8: now also GPIO2.4; no longer GPIO.14
- net RB9: now also GPIO2.5; no longer GPIO.12
Other:
- moved on the sheet: RES4
